File: Rechargable 5V power bank REV 0.5/Rechargable 5V power bank REV 0.5.sch (KiCad schematic (older format))
At the start: 63 parts, among them J1 Micro_USB_CONN, J2 USB-A_CONN, J3 1POS_CONN_PAD_30X30MM_H1MM, J4 1POS_CONN_PAD_30X30MM_H1MM, J5 1POS_CONN_PAD_30X30MM_H1MM, J6 1POS_CONN_PAD_30X30MM_H1MM, Q1 NMOS_20V_3.6A_SOT-23-3, Q2 NMOS_20V_3.6A_SOT-23-3, Q3 PMOS_20V_4.2A_SOT-23-3, U1 BQ24090DGQR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

Commit message: UPLOAD REV 0.5
Parts:
- removed BT1: 18650 Li-ion Battery Cell, symbol Device:Battery_Cell
- removed TP1, TP10, TP11, TP2, TP3, TP4, TP5, TP6, TP7, TP8, TP9: TP_12.5X12.5_MM, symbol TESTPOINTS:TP_12.5X12.5_MM
- added BAT1: BAT_18650_HOLDER_SMD, BATTERIES:BAT_18650_HOLDER_SMD, symbol BATTERIES:BAT_18650_HOLDER_SMD
- added TP1, TP10, TP11, TP2, TP3, TP4, TP5, TP6, TP7, TP8, TP9: TP_1.25X1.25_MM, TESTPOINTS:TP_RECT_1.25X1.25, symbol TESTPOINTS:TP_1.25X1.25_MM
- C1, C10, C11, C2, C3, C6, C8, C9: footprint Capacitor_SMD:C_0603_1608Metric_Pad1.05x0.95mm_HandSolder -> CAPACITORS:CACP_0603_HandSolder
- C4, C7: footprint Capacitor_SMD:C_1210_3225Metric_Pad1.42x2.65mm_HandSolder -> CAPACITORS:CAPC_1210_HandSolder
- C5: footprint Capacitor_SMD:C_0805_2012Metric_Pad1.15x1.40mm_HandSolder -> CAPACITORS:CAPC_0805_HandSolder
- D1, D4: footprint (none) -> DIODES:DO-214AC
- D2, D3: footprint (none) -> DIODES:DO-214AB
- DS1, DS2: footprint LED_SMD:LED_0603_1608Metric_Pad1.05x0.95mm_HandSolder -> LEDS:LEDC_0603_HandSolder
- F1: footprint (none) -> FUSES:POLYFUSEC_1812
- J1: footprint (none) -> CONNECTORS:USB-TYPE-B_CONN_PORT; Link https://www.digikey.com/product-detail/en/adam-tech/MCR-B-S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 -> https://www.digikey.com/product-detail/en/molex/0475890001/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; Manufacturer Adam Tech -> Molex; Manufacturer_PN MCR-B-S-RA-SMT-EH4B-T/R -> 0475890001; Price for 1 0.37000 -> 0.78000; Price for 100 0.24480 -> 0.58810; VAL MicroUSB connector -> Micro_USB_CONN
- J2: footprint (none) -> CONNECTORS:USB-TYPE-A_CONN_PORT
- J3, J4, J5, J6: footprint (none) -> PADS:PAD_RECT_30X30; ASSEMBLY N/A -> NO; BOM_IGNORE N/A -> YES
- L1: footprint (none) -> INDUCTORS:CDRH104R
- NTC1: footprint (none) -> RESISTORS:RESC_0603_HandSolder
- Q1, Q2, Q3: footprint (none) -> TRANSISTORS:SOT-23_Handsoldering
- R1, R10, R11, R12, R13, R14, R19, R2, R3, R4, R5, R6, R7, R8, R9: footprint Resistor_SMD:R_0603_1608Metric_Pad1.05x0.95mm_HandSolder -> RESISTORS:RESC_0603_HandSolder
- R15, R16, R17, R18: footprint Resistor_SMD:R_0603_1608Metric_Pad1.05x0.95mm_HandSolder -> RESISTORS:RESC_0603_HandSolder; ASSEMBLY N/A -> NO; BOM_IGNORE N/A -> YES
- U1: footprint (none) -> ICs:BQ24090DGQR_MSOP-10
- U2: footprint Package_TO_SOT_SMD:SOT-23-6_Handsoldering -> ICs:AP9101C_SOT-23-6_Handsoldering
- U3: footprint (none) -> ICs:PAM2421_SOIC-8-EP
Connections:
- wire segments 191 -> 195
Other:
- note added: "0.5"
- note added: "7-Aug-2020"
- note removed: "0.3"
- note removed: "7-Jul-2020"
