File: Rechargeable 5V power bank REV 0.5/Rechargeable 5V power bank REV 0.5.sch (KiCad schematic (older format))
At the start: 63 parts, among them J1 Micro_USB_CONN, J2 USB-A_CONN, J3 1POS_CONN_PAD_30X30MM_H1MM, J4 1POS_CONN_PAD_30X30MM_H1MM, J5 1POS_CONN_PAD_30X30MM_H1MM, J6 1POS_CONN_PAD_30X30MM_H1MM, Q1 NMOS_20V_3.6A_SOT-23-3, Q2 NMOS_20V_3.6A_SOT-23-3, Q3 PMOS_20V_4.2A_SOT-23-3, U1 BQ24090DGQR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

Commit message: Update and minor fix
Parts:
- R15, R16, R17, R18: ASSEMBLY N/A -> NO; BOM_IGNORE N/A -> YES
Other:
- note added: "Rechargeable 5V power bank"
Changed lines of the file:
@@
 Wire Wire Line
 	3550 7750 3550 7900
-$Comp
-L RESISTORS:RESC_10K_0603 R15
-U 1 1 5F32E18B
-P 3550 7650
-AR Path="/5F32E18B" Ref="R15"  Part="1"
-AR Path="/5F0383B8/5F32E18B" Ref="R?"  Part="1"
-F 0 "R15" H 3500 7500 50  0000 C CNN
-F 1 "RESC_10K_0603" H 4500 8550 50  0001 L CNN
-F 2 "RESISTORS:RESC_0603_HandSolder" H 3600 8850 50  0001 C CNN
-F 3 "https://www.seielect.com/catalog/sei-rncp.pdf" H 3550 7650 50  0001 C CNN
-F 4 "10K" H 3450 7800 50  0000 C CNN "VAL"
-F 5 "RNCP0603FTD10K0" H 3600 8850 50  0001 C CNN "Manufacturer_PN"
-F 6 "Stackpole Electronics Inc" H 3800 8750 50  0001 C CNN "Manufacturer"
-F 7 "0.1" H 3600 8750 50  0001 C CNN "Price for 1"
-F 8 "0.02730" H 3800 8750 50  0001 C CNN "Price for 100"
-F 9 "https://www.digikey.com/product-detail/en/stackpole-electronics-inc/RNCP0603FTD10K0/RNCP0603FTD10K0CT-ND/2240478" H 3600 8850 50  0001 C CNN "Link"
-F 10 "N/A" H 3350 8750 50  0001 C CNN "ASSEMBLY"
-F 11 "N/A" H 3400 8850 50  0001 C CNN "BOM_IGNORE"
-	1    3550 7650
-	-1   0    0    1
-$EndComp
-$Comp
-L RESISTORS:RESC_10K_0603 R18
-U 1 1 5F32E199
-P 3900 8300
-AR Path="/5F32E199" Ref="R18"  Part="1"
-AR Path="/5F0383B8/5F32E199" Ref="R?"  Part="1"
-F 0 "R18" H 3850 8150 50  0000 C CNN
-F 1 "RESC_10K_0603" H 4850 9200 50  0001 L CNN
-F 2 "RESISTORS:RESC_0603_HandSolder" H 3950 9500 50  0001 C CNN
-F 3 "https://www.seielect.com/catalog/sei-rncp.pdf" H 3900 8300 50  0001 C CNN
-F 4 "10K" H 3800 8450 50  0000 C CNN "VAL"
-F 5 "RNCP0603FTD10K0" H 3950 9500 50  0001 C CNN "Manufacturer_PN"
-F 6 "Stackpole Electronics Inc" H 4150 9400 50  0001 C CNN "Manufacturer"
-F 7 "0.1" H 3950 9400 50  0001 C CNN "Price for 1"
-F 8 "0.02730" H 4150 9400 50  0001 C CNN "Price for 100"
-F 9 "https://www.digikey.com/product-detail/en/stackpole-electronics-inc/RNCP0603FTD10K0/RNCP0603FTD10K0CT-ND/2240478" H 3950 9500 50  0001 C CNN "Link"
-F 10 "N/A" H 3700 9400 50  0001 C CNN "ASSEMBLY"
-F 11 "N/A" H 3750 9500 50  0001 C CNN "BOM_IGNORE"
-	1    3900 8300
-	-1   0    0    1
-$EndComp
-$Comp
-L RESISTORS:RESC_10K_0603 R17
-U 1 1 5F32E1A7
-P 3550 8300
-AR Path="/5F32E1A7" Ref="R17"  Part="1"
-AR Path="/5F0383B8/5F32E1A7" Ref="R?"  Part="1"
-F 0 "R17" H 3500 8150 50  0000 C CNN
-F 1 "RESC_10K_0603" H 4500 9200 50  0001 L CNN
-F 2 "RESISTORS:RESC_0603_HandSolder" H 3600 9500 50  0001 C CNN
-F 3 "https://www.seielect.com/catalog/sei-rncp.pdf" H 3550 8300 50  0001 C CNN
-F 4 "10K" H 3450 8450 50  0000 C CNN "VAL"
-F 5 "RNCP0603FTD10K0" H 3600 9500 50  0001 C CNN "Manufacturer_PN"
-F 6 "Stackpole Electronics Inc" H 3800 9400 50  0001 C CNN "Manufacturer"
-F 7 "0.1" H 3600 9400 50  0001 C CNN "Price for 1"
-F 8 "0.02730" H 3800 9400 50  0001 C CNN "Price for 100"
-F 9 "https://www.digikey.com/product-detail/en/stackpole-electronics-inc/RNCP0603FTD10K0/RNCP0603FTD10K0CT-ND/2240478" H 3600 9500 50  0001 C CNN "Link"
-F 10 "N/A" H 3350 9400 50  0001 C CNN "ASSEMBLY"
-F 11 "N/A" H 3400 9500 50  0001 C CNN "BOM_IGNORE"
-	1    3550 8300
-	-1   0    0    1
-$EndComp
 Wire Wire Line
 	4600 8000 4350 8000
@@
 Connectors
 Text Notes 5750 950  0    200  ~ 0
-Rechargable 5[V] power bank
+Rechargeable 5V power bank
 Text Notes 6400 6800 0    200  ~ 0
 Test points
@@
 AR Path="/5F32E37B" Ref="R16"  Part="1"
 AR Path="/5F0383B8/5F32E37B" Ref="R?"  Part="1"
-F 0 "R16" H 3850 7500 50  0000 C CNN
+F 0 "R16" H 3800 7500 50  0000 C CNN
 F 1 "RESC_10K_0603" H 4850 8550 50  0001 L CNN
 F 2 "RESISTORS:RESC_0603_HandSolder" H 3950 8850 50  0001 C CNN
@@
 F 8 "0.02730" H 4150 8750 50  0001 C CNN "Price for 100"
 F 9 "https://www.digikey.com/product-detail/en/stackpole-electronics-inc/RNCP0603FTD10K0/RNCP0603FTD10K0CT-ND/2240478" H 3950 8850 50  0001 C CNN "Link"
-F 10 "N/A" H 3700 8750 50  0001 C CNN "ASSEMBLY"
-F 11 "N/A" H 3750 8850 50  0001 C CNN "BOM_IGNORE"
+F 10 "NO" H 3700 8750 50  0001 C CNN "ASSEMBLY"
+F 11 "YES" H 3750 8850 50  0001 C CNN "BOM_IGNORE"
 	1    3900 7650
 	-1   0    0    1
@@
 Text Notes 3500 7850 0    100  ~ 0
 X\nNC\n
-Text Notes 3500 8500 0    100  ~ 0
-X\nNC\n
 Text Notes 3850 8500 0    100  ~ 0
 X\nNC\n
@@
 	1    0    0    -1
 $EndComp
+$Comp
+L RESISTORS:RESC_10K_0603 R15
+U 1 1 5F2ED0DD
+P 3550 7650
+AR Path="/5F2ED0DD" Ref="R15"  Part="1"
+AR Path="/5F0383B8/5F2ED0DD" Ref="R?"  Part="1"
+F 0 "R15" H 3450 7500 50  0000 C CNN
+F 1 "RESC_10K_0603" H 4500 8550 50  0001 L CNN
+F 2 "RESISTORS:RESC_0603_HandSolder" H 3600 8850 50  0001 C CNN
+F 3 "https://www.seielect.com/catalog/sei-rncp.pdf" H 3550 7650 50  0001 C CNN
+F 4 "10K" H 3450 7800 50  0000 C CNN "VAL"
+F 5 "RNCP0603FTD10K0" H 3600 8850 50  0001 C CNN "Manufacturer_PN"
+F 6 "Stackpole Electronics Inc" H 3800 8750 50  0001 C CNN "Manufacturer"
+F 7 "0.1" H 3600 8750 50  0001 C CNN "Price for 1"
+F 8 "0.02730" H 3800 8750 50  0001 C CNN "Price for 100"
+F 9 "https://www.digikey.com/product-detail/en/stackpole-electronics-inc/RNCP0603FTD10K0/RNCP0603FTD10K0CT-ND/2240478" H 3600 8850 50  0001 C CNN "Link"
+F 10 "NO" H 3350 8750 50  0001 C CNN "ASSEMBLY"
+F 11 "YES" H 3400 8850 50  0001 C CNN "BOM_IGNORE"
+	1    3550 7650
+	-1   0    0    1
+$EndComp
+$Comp
+L RESISTORS:RESC_10K_0603 R17
+U 1 1 5F2EE1BA
+P 3550 8300
+AR Path="/5F2EE1BA" Ref="R17"  Part="1"
+AR Path="/5F0383B8/5F2EE1BA" Ref="R?"  Part="1"
+F 0 "R17" H 3450 8150 50  0000 C CNN
+F 1 "RESC_10K_0603" H 4500 9200 50  0001 L CNN
+F 2 "RESISTORS:RESC_0603_HandSolder" H 3600 9500 50  0001 C CNN
+F 3 "https://www.seielect.com/catalog/sei-rncp.pdf" H 3550 8300 50  0001 C CNN
+F 4 "10K" H 3450 8450 50  0000 C CNN "VAL"
+F 5 "RNCP0603FTD10K0" H 3600 9500 50  0001 C CNN "Manufacturer_PN"
+F 6 "Stackpole Electronics Inc" H 3800 9400 50  0001 C CNN "Manufacturer"
+F 7 "0.1" H 3600 9400 50  0001 C CNN "Price for 1"
+F 8 "0.02730" H 3800 9400 50  0001 C CNN "Price for 100"
+F 9 "https://www.digikey.com/product-detail/en/stackpole-electronics-inc/RNCP0603FTD10K0/RNCP0603FTD10K0CT-ND/2240478" H 3600 9500 50  0001 C CNN "Link"
+F 10 "NO" H 3350 9400 50  0001 C CNN "ASSEMBLY"
+F 11 "YES" H 3400 9500 50  0001 C CNN "BOM_IGNORE"
+	1    3550 8300
+	-1   0    0    1
+$EndComp
+$Comp
+L RESISTORS:RESC_10K_0603 R18
+U 1 1 5F2EEA92
+P 3900 8300
+AR Path="/5F2EEA92" Ref="R18"  Part="1"
+AR Path="/5F0383B8/5F2EEA92" Ref="R?"  Part="1"
+F 0 "R18" H 3800 8150 50  0000 C CNN
+F 1 "RESC_10K_0603" H 4850 9200 50  0001 L CNN
+F 2 "RESISTORS:RESC_0603_HandSolder" H 3950 9500 50  0001 C CNN
+F 3 "https://www.seielect.com/catalog/sei-rncp.pdf" H 3900 8300 50  0001 C CNN
+F 4 "10K" H 3800 8450 50  0000 C CNN "VAL"
+F 5 "RNCP0603FTD10K0" H 3950 9500 50  0001 C CNN "Manufacturer_PN"
+F 6 "Stackpole Electronics Inc" H 4150 9400 50  0001 C CNN "Manufacturer"
+F 7 "0.1" H 3950 9400 50  0001 C CNN "Price for 1"
+F 8 "0.02730" H 4150 9400 50  0001 C CNN "Price for 100"
+F 9 "https://www.digikey.com/product-detail/en/stackpole-electronics-inc/RNCP0603FTD10K0/RNCP0603FTD10K0CT-ND/2240478" H 3950 9500 50  0001 C CNN "Link"
+F 10 "NO" H 3700 9400 50  0001 C CNN "ASSEMBLY"
+F 11 "YES" H 3750 9500 50  0001 C CNN "BOM_IGNORE"
+	1    3900 8300
+	-1   0    0    1
+$EndComp
+Text Notes 3500 8500 0    100  ~ 0
+X\nNC\n
 $EndSCHEMATC
